File: Airhockeypuck.sch (EAGLE design)
At the start: 23 parts, among them J1 USB-MB-H

Commit message: minor edits
Connections:
- net +3V3: now also U$10.2.VIN
- net B2: now also U$10.4.SDA
- net B3: now also U$10.5.SCL
- net GND: now also U$10.3.GND

Commit message: minor edits
Parts:
- added U$11: HC-08, MEE_433:HC-08
- U$6, U$7: value CONN_08 -> DRV8835; device MEE_433:CONN_08 -> MEE_433:DRV8835
Connections:
- new net N$10: U$6.10.BENABLE
- new net N$11: U$6.11.BPHASE
- new net N$12: U$6.12.AENABLE
- new net N$13: U$6.13.APHASE
- new net N$14: U$11.4.RX
- new net N$16: U$7.10.BENABLE
- new net N$17: U$7.11.BPHASE
- new net N$18: U$7.12.AENABLE
- new net N$19: U$7.13.APHASE
- new net N$3: U$11.1.VCC
- new net N$9: U$11.3.TX
- net +3V3: now also U$6.9.VCC, U$7.9.VCC; no longer U$7.2
- net +5V: no longer U$6.2
- net A0: no longer U$7.8
- net A1: no longer U$7.7
- net A4/LED: no longer U$7.3
- net B13: no longer U$6.6
- net B14: no longer U$6.7
- net B15: no longer U$6.8
- net B2: no longer U$7.6
- net B3: no longer U$7.5
- net B4/USER: no longer U$7.4
- net B7: no longer U$6.3
- net B8: no longer U$6.4
- net B9: no longer U$6.5
- net GND: now also U$11.2.GND, U$6.8.GND, U$7.8.GND; no longer U$6.1, U$7.1
Other:
- moved on the sheet: U$2
