File: Airhockeypuck.brd (EAGLE design)
At the start: 80 x 80 mm, 24 parts, among them J1 USB-MB-H

Commit message: error-checking passed
Routing:
- net B14: track 9.68 -> 12.6 mm
- net +3V3: track 255.8 -> 254.3 mm, vias 11 -> 10
- net D+: track 77.5 -> 76.2 mm
- net B2: track 35.3 -> 34.1 mm
- net +5V: track 68.1 -> 67.4 mm
Changed lines of the file:
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@@
 <wire x1="15.24" y1="21.59" x2="15.24" y2="22.86" width="0.1524" layer="1"/>
 <wire x1="20.32" y1="27.94" x2="20.32" y2="33.02" width="0.1524" layer="1"/>
-<wire x1="20.32" y1="33.02" x2="17.589" y2="35.751" width="0.1524" layer="1"/>
-<wire x1="17.589" y1="35.751" x2="13.2811875" y2="37.759765625" width="0.1524" layer="1"/>
-<wire x1="13.2811875" y1="37.759765625" x2="12.95935625" y2="37.846" width="0.1524" layer="1"/>
 <wire x1="15.24" y1="22.86" x2="20.32" y2="27.94" width="0.1524" layer="1"/>
-<wire x1="-6.35" y1="33.02" x2="-8.89" y2="35.56" width="0.1524" layer="16"/>
-<wire x1="-8.89" y1="35.56" x2="-5.08" y2="39.37" width="0.1524" layer="1"/>
-<wire x1="-5.08" y1="39.37" x2="1.524" y2="39.37" width="0.1524" layer="1"/>
+<wire x1="1.524" y1="39.37" x2="-5.08" y2="39.37" width="0.1524" layer="1"/>
 <wire x1="-19.937765625" y1="27.078584375" x2="-19.911415625" y2="27.078584375" width="0.1524" layer="1"/>
 <wire x1="-19.911415625" y1="27.078584375" x2="-19.05" y2="27.94" width="0.1524" layer="1"/>
@@
 <via x="-16.51" y="29.21" extent="1-16" drill="0.35"/>
 <wire x1="-16.51" y1="29.21" x2="-15.24" y2="29.21" width="0.1524" layer="1"/>
-<wire x1="12.95935625" y1="37.846" x2="7.271715625" y2="39.37" width="0.1524" layer="1"/>
-<wire x1="7.271715625" y1="39.37" x2="3.81" y2="39.37" width="0.1524" layer="1"/>
 <wire x1="3.81" y1="39.37" x2="3.048" y2="38.608" width="0.1524" layer="1"/>
 <wire x1="3.048" y1="38.608" x2="3.048" y2="37.846" width="0.1524" layer="1"/>
 <wire x1="-15.24" y1="29.21" x2="-15.24" y2="31.75" width="0.1524" layer="1"/>
 <via x="-15.24" y="31.75" extent="1-16" drill="0.35"/>
-<wire x1="-15.24" y1="31.75" x2="-13.97" y2="33.02" width="0.1524" layer="16"/>
-<wire x1="-13.97" y1="33.02" x2="-10.16" y2="33.02" width="0.1524" layer="16"/>
-<via x="-10.16" y="33.02" extent="1-16" drill="0.35"/>
-<wire x1="-10.16" y1="33.02" x2="-6.35" y2="33.02" width="0.1524" layer="16"/>
-<via x="-8.89" y="35.56" extent="1-16" drill="0.35"/>
+<wire x1="-11.43" y1="31.75" x2="-15.24" y2="31.75" width="0.1524" layer="16"/>
+<via x="-11.43" y="31.75" extent="1-16" drill="0.35"/>
 <via x="11.43" y="-19.05" extent="1-16" drill="0.35"/>
 <via x="6.096" y="-14.986" extent="1-16" drill="0.35"/>
+<wire x1="20.32" y1="33.02" x2="17.589" y2="35.751" width="0.1524" layer="1"/>
+<wire x1="7.271715625" y1="39.37" x2="3.81" y2="39.37" width="0.1524" layer="1"/>
+<wire x1="17.589" y1="35.751" x2="14.759828125" y2="37.070265625" width="0.1524" layer="1"/>
+<wire x1="9.57145" y1="37.070265625" x2="7.271715625" y2="39.37" width="0.1524" layer="1"/>
+<wire x1="14.759828125" y1="37.070265625" x2="9.57145" y2="37.070265625" width="0.1524" layer="1"/>
+<wire x1="-5.08" y1="39.37" x2="-6.35" y2="38.1" width="0.1524" layer="1"/>
+<wire x1="-6.35" y1="38.1" x2="-6.35" y2="33.02" width="0.1524" layer="1"/>
+<wire x1="-11.43" y1="31.75" x2="-7.62" y2="31.75" width="0.1524" layer="1"/>
+<wire x1="-7.62" y1="31.75" x2="-6.35" y2="33.02" width="0.1524" layer="1"/>
 </signal>
 <signal name="N$2">
@@
 <wire x1="33.02" y1="-13.97" x2="36.83" y2="-10.16" width="0.1524" layer="1"/>
 <wire x1="36.83" y1="-10.16" x2="36.83" y2="-7.62" width="0.1524" layer="1"/>
-<wire x1="27.94" y1="1.27" x2="27.94" y2="27.94" width="0.1524" layer="1"/>
-<wire x1="27.94" y1="27.94" x2="26.67" y2="29.21" width="0.1524" layer="1"/>
+<wire x1="27.94" y1="1.27" x2="27.94" y2="26.67" width="0.1524" layer="1"/>
+<wire x1="27.94" y1="26.67" x2="25.4" y2="29.21" width="0.1524" layer="1"/>
 <wire x1="33.02" y1="-19.01575625" x2="33.02" y2="-13.97" width="0.1524" layer="1"/>
 <wire x1="36.83" y1="-7.62" x2="27.94" y2="1.27" width="0.1524" layer="1"/>
-<via x="26.67" y="29.21" extent="1-16" drill="0.35"/>
-<wire x1="26.67" y1="29.21" x2="19.05" y2="29.21" width="0.1524" layer="16"/>
+<via x="25.4" y="29.21" extent="1-16" drill="0.35"/>
+<wire x1="25.4" y1="29.21" x2="19.05" y2="29.21" width="0.1524" layer="16"/>
 <via x="19.05" y="29.21" extent="1-16" drill="0.35"/>
 <wire x1="19.05" y1="29.21" x2="17.78" y2="29.21" width="0.1524" layer="1"/>
@@
 <via x="3.81" y="35.56" extent="1-16" drill="0.35"/>
 <wire x1="-13.97" y1="34.29" x2="-11.43" y2="34.29" width="0.1524" layer="16"/>
-<wire x1="-10.16" y1="35.56" x2="3.81" y2="35.56" width="0.1524" layer="16"/>
 <wire x1="3.81" y1="35.56" x2="5.588" y2="37.338" width="0.1524" layer="1"/>
 <wire x1="5.588" y1="37.338" x2="5.588" y2="37.846" width="0.1524" layer="1"/>
+<wire x1="-10.16" y1="35.56" x2="3.81" y2="35.56" width="0.1524" layer="16"/>
 </signal>
 <signal name="A0">
@@
 <contactref element="U$1" pad="6"/>
 <contactref element="U$10" pad="4."/>
-<wire x1="1.016" y1="-8.636" x2="0.762" y2="-8.89" width="0.1524" layer="1"/>
-<wire x1="0.762" y1="-8.89" x2="0" y2="-8.89" width="0.1524" layer="1"/>
 <wire x1="1.016" y1="-8.636" x2="0" y2="-7.62" width="0.1524" layer="1"/>
 <wire x1="0" y1="-7.62" x2="0" y2="-5.08" width="0.1524" layer="1"/>
@@
 <contactref element="U$1" pad="25"/>
 <contactref element="U$11" pad="4.RX"/>
-<wire x1="-11.629690625" y1="33.219690625" x2="-11.629690625" y2="37.2305875" width="0.1524" layer="1"/>
-<wire x1="-7.62" y1="29.21" x2="-11.629690625" y2="33.219690625" width="0.1524" layer="1"/>
+<wire x1="-7.62" y1="29.21" x2="-9.398" y2="30.988" width="0.1524" layer="1"/>
+<wire x1="-12.7" y1="30.988" x2="-12.827" y2="31.115" width="0.1524" layer="1"/>
+<wire x1="-12.827" y1="31.115" x2="-12.827" y2="35.433" width="0.1524" layer="1"/>
+<wire x1="-11.629690625" y1="36.630309375" x2="-11.629690625" y2="37.2305875" width="0.1524" layer="1"/>
+<wire x1="-9.398" y1="30.988" x2="-12.7" y2="30.988" width="0.1524" layer="1"/>
+<wire x1="-12.827" y1="35.433" x2="-11.629690625" y2="36.630309375" width="0.1524" layer="1"/>
 </signal>
 <signal name="B13">
@@
 <wire x1="20.574" y1="14.605" x2="20.701" y2="14.605" width="0.1524" layer="1"/>
 <wire x1="20.701" y1="14.605" x2="20.701" y2="25.4" width="0.1524" layer="1"/>
-<wire x1="20.701" y1="25.4" x2="20.5105" y2="25.5905" width="0.1524" layer="1"/>
-<wire x1="20.5105" y1="25.5905" x2="20.32" y2="25.781" width="0.1524" layer="1"/>
 <wire x1="16.129" y1="25.781" x2="15.24" y2="26.67" width="0.1524" layer="1"/>
 <wire x1="15.24" y1="26.67" x2="15.24" y2="29.21" width="0.1524" layer="1"/>
-<wire x1="20.5105" y1="25.5905" x2="20.4907" y2="25.5905" width="0.1524" layer="1"/>
-<wire x1="20.4907" y1="25.5905" x2="20.32" y2="25.7612" width="0.1524" layer="1"/>
 <via x="20.32" y="25.7612" extent="1-16" drill="0.35"/>
 <wire x1="20.32" y1="25.7612" x2="16.7838" y2="25.7612" width="0.1524" layer="16"/>
@@
 <wire x1="8.89" y1="-1.27" x2="7.62" y2="-2.54" width="0.1524" layer="1"/>
 <wire x1="7.62" y1="-2.54" x2="7.62" y2="-3.81" width="0.1524" layer="1"/>
+<wire x1="20.701" y1="25.4" x2="20.3398" y2="25.7612" width="0.1524" layer="1"/>
+<wire x1="20.3398" y1="25.7612" x2="20.32" y2="25.7612" width="0.1524" layer="1"/>
 </signal>
 <signal name="D+">
@@
 <wire x1="30.48" y1="21.59" x2="26.67" y2="21.59" width="0.1524" layer="16"/>
 <via x="26.67" y="21.59" extent="1-16" drill="0.35"/>
-<wire x1="26.67" y1="21.59" x2="26.67" y2="27.94" width="0.1524" layer="1"/>
-<wire x1="26.67" y1="27.94" x2="21.59" y2="33.02" width="0.1524" layer="1"/>
 <via x="21.59" y="33.02" extent="1-16" drill="0.35"/>
 <wire x1="21.59" y1="33.02" x2="19.05" y2="33.02" width="0.1524" layer="16"/>
 <via x="19.05" y="33.02" extent="1-16" drill="0.35"/>
 <wire x1="19.05" y1="33.02" x2="7.62" y2="33.02" width="0.1524" layer="1"/>
-<wire x1="2.54" y1="30.48" x2="2.54" y2="29.21" width="0.1524" layer="1"/>
 <wire x1="7.62" y1="33.02" x2="6.35" y2="34.29" width="0.1524" layer="1"/>
 <wire x1="6.35" y1="34.29" x2="3.81" y2="34.29" width="0.1524" layer="1"/>
 <wire x1="3.81" y1="34.29" x2="2.54" y2="33.02" width="0.1524" layer="1"/>
+<wire x1="26.67" y1="21.59" x2="26.67" y2="26.67" width="0.1524" layer="1"/>
+<wire x1="26.67" y1="26.67" x2="22.86" y2="30.48" width="0.1524" layer="1"/>
+<wire x1="22.86" y1="30.48" x2="22.86" y2="31.75" width="0.1524" layer="1"/>
+<wire x1="22.86" y1="31.75" x2="21.59" y2="33.02" width="0.1524" layer="1"/>
 <wire x1="2.54" y1="33.02" x2="2.54" y2="29.21" width="0.1524" layer="1"/>
 </signal>
@@
 <wire x1="26.67" y1="-23.1867" x2="26.371896875" y2="-23.484803125" width="0.1524" layer="1"/>
 <wire x1="26.246740625" y1="-10.583259375" x2="24.13" y2="-12.7" width="0.1524" layer="1"/>
-<wire x1="26.9604375" y1="-10.583259375" x2="27.093259375" y2="-10.583259375" width="0.1524" layer="1"/>
 </signal>
 <signal name="A4">
